File: Rev. 0/Eagle/C64_CHARSETSw_4k.brd (EAGLE design)
At the start: 22 x 45 mm, 12 parts, among them IC1 M27C512-DIP28, IC2 2332

Commit message: Silk Screen Revision
Parts:
- added U$11: (no value), Logo:SVEN_TAG
- added U$6: OPEN_SOURCE_HW, Logo:OPENHW
Other:
- board text added: "4x10k"
- board text added: "http://github.com/ svenpetersen1965"
Changed lines of the file:
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@@
 <?xml version="1.0" encoding="utf-8"?>
 <!DOCTYPE eagle SYSTEM "eagle.dtd">
-<eagle version="9.2.2">
+<eagle version="9.5.2">
 <drawing>
 <settings>
@@
 <layer number="19" name="Unrouted" color="6" fill="1" visible="yes" active="yes"/>
 <layer number="20" name="Dimension" color="24" fill="1" visible="yes" active="yes"/>
-<layer number="21" name="tPlace" color="7" fill="1" visible="no" active="yes"/>
+<layer number="21" name="tPlace" color="7" fill="1" visible="yes" active="yes"/>
 <layer number="22" name="bPlace" color="7" fill="1" visible="yes" active="yes"/>
 <layer number="23" name="tOrigins" color="15" fill="1" visible="yes" active="yes"/>
 <layer number="24" name="bOrigins" color="15" fill="1" visible="yes" active="yes"/>
 <layer number="25" name="tNames" color="7" fill="1" visible="yes" active="yes"/>
-<layer number="26" name="bNames" color="7" fill="1" visible="no" active="yes"/>
+<layer number="26" name="bNames" color="7" fill="1" visible="yes" active="yes"/>
 <layer number="27" name="tValues" color="7" fill="1" visible="no" active="yes"/>
 <layer number="28" name="bValues" color="7" fill="1" visible="no" active="yes"/>
@@
 <layer number="45" name="Holes" color="7" fill="1" visible="no" active="yes"/>
 <layer number="46" name="Milling" color="3" fill="1" visible="no" active="yes"/>
-<layer number="47" name="Measures" color="7" fill="1" visible="no" active="yes"/>
+<layer number="47" name="Measures" color="7" fill="1" visible="yes" active="yes"/>
 <layer number="48" name="Document" color="5" fill="1" visible="yes" active="yes"/>
 <layer number="49" name="Reference" color="7" fill="1" visible="yes" active="yes"/>
 <layer number="50" name="dxf" color="7" fill="1" visible="no" active="no"/>
-<layer number="51" name="tDocu" color="7" fill="1" visible="no" active="yes"/>
+<layer number="51" name="tDocu" color="7" fill="1" visible="yes" active="yes"/>
 <layer number="52" name="bDocu" color="7" fill="1" visible="no" active="yes"/>
 <layer number="53" name="tGND_GNDA" color="7" fill="1" visible="no" active="no"/>
@@
 <layer number="250" name="Descript" color="7" fill="1" visible="no" active="no"/>
 <layer number="251" name="SMDround" color="7" fill="1" visible="no" active="no"/>
+<layer number="252" name="BR-BS" color="7" fill="1" visible="no" active="yes"/>
+<layer number="253" name="BR-LS" color="7" fill="1" visible="no" active="yes"/>
 <layer number="254" name="OrgLBR" color="7" fill="1" visible="no" active="no"/>
 <layer number="255" name="Accent" color="7" fill="1" visible="yes" active="yes"/>
@@
 C64 short board</text>
 <text x="11.27125" y="3.81" size="1.1684" layer="47" ratio="12" rot="R90">Rev. 0</text>
-<text x="11.90625" y="3.81" size="1.1684" layer="21" ratio="12" rot="R90">CHARSET Adapt/
+<text x="9.36625" y="3.96875" size="1.016" layer="21" ratio="12" rot="R90">CHARSET Adapt/
 Switch C64</text>
-<text x="13.97" y="3.81" size="1.1684" layer="21" ratio="12" rot="R90">Rev. 0</text>
+<text x="10.795" y="3.96875" size="1.016" layer="21" ratio="12" rot="R90">Rev. 0</text>
 <text x="9.8425" y="4.7625" size="1.778" layer="22" ratio="12" rot="MR90">C64 CHARSET Adaptor/
 Switch Rev. 0</text>
@@
 <wire x1="17.78" y1="38.57625" x2="18.415" y2="38.57625" width="0.127" layer="21"/>
 <text x="21.2725" y="37.94125" size="1.016" layer="21" rot="R90">GND</text>
+<text x="6.6675" y="34.6075" size="1.016" layer="21">4x10k</text>
+<text x="15.39875" y="3.96875" size="1.016" layer="21" rot="R90">http://github.com/
+svenpetersen1965</text>
+<text x="15.5575" y="36.5125" size="1.016" layer="22" rot="MR0" align="bottom-center">GND</text>
+<wire x1="11.7475" y1="37.62375" x2="11.7475" y2="36.98875" width="0.127" layer="22"/>
+<wire x1="11.7475" y1="36.98875" x2="13.97" y2="36.98875" width="0.127" layer="22"/>
+<wire x1="16.98625" y1="36.98875" x2="19.3675" y2="36.98875" width="0.127" layer="22"/>
+<wire x1="19.3675" y1="36.98875" x2="19.3675" y2="37.62375" width="0.127" layer="22"/>
+<wire x1="8.255" y1="41.275" x2="7.62" y2="41.275" width="0.127" layer="22"/>
+<wire x1="7.62" y1="41.275" x2="7.62" y2="38.57625" width="0.127" layer="22"/>
+<wire x1="7.62" y1="38.57625" x2="8.255" y2="38.57625" width="0.127" layer="22"/>
+<text x="7.3025" y="39.84625" size="1.016" layer="22" rot="MR270" align="bottom-center">+5V</text>
 </plain>
 <attributes>
@@
 </element>
 <element name="R2" library="SMD" package="0805" value="10k" x="13.6525" y="29.845" smashed="yes" rot="R180">
-<attribute name="NAME" x="13.58775" y="27.6185" size="1.016" layer="25" ratio="10"/>
+<attribute name="NAME" x="11.68275" y="27.6185" size="1.016" layer="25" ratio="10"/>
 <attribute name="VALUE" x="15.24" y="30.2895" size="1.016" layer="27" ratio="10" rot="R180"/>
 </element>
@@
 </element>
 <element name="R1" library="SMD" package="0805" value="10k" x="8.73125" y="29.845" smashed="yes">
-<attribute name="NAME" x="8.03275" y="27.84475" size="1.016" layer="25" ratio="10"/>
+<attribute name="NAME" x="7.874" y="27.686" size="1.016" layer="25" ratio="10"/>
 <attribute name="VALUE" x="7.14375" y="29.4005" size="1.016" layer="27" ratio="10"/>
 </element>
+<element name="U$6" library="Logo" package="OPENHW" value="OPEN_SOURCE_HW" x="15.5575" y="20.16125" smashed="yes" rot="R90"/>
+<element name="U$11" library="Logo" package="SVEN_TAG" value="" x="7.9375" y="10.795" smashed="yes" rot="MR0"/>
 </elements>
 <signals>
